File: Circuit/bbesc_kiCad.kicad_pcb (KiCad board)
At the start: 2 copper layers, 110.5 x 82.5 mm, 82 parts, among them J1 CONN_01X02, J10 CONN_01X01, J11 CONN_01X01, J12 CONN_01X01, J13 CONN_01X01, J14 CONN_01X01, J15 CONN_01X02, J16 CONN_01X02, J17 CONN_01X01, J18 CONN_01X01, J19 CONN_01X01, J2 CONN_01X06, J3 CONN_01X06, J4 CONN_01X06, J5 CONN_01X02, J6 CONN_01X02, J7 CONN_01X01, J8 CONN_01X01, J9 RJ45, Q1 Q_NMOS_GDS, Q2 Q_NMOS_GDS, Q3 Q_NMOS_GDS, Q4 Q_NMOS_GDS, Q5 Q_NMOS_GDS, Q6 Q_NMOS_GDS, U1 teensy_3-2, U2 IR2101, U3 IR2101, U4 IR2101, U5 LM324N, U6 LM7805

Commit message: mv to linux
Routing:
- net Net-(R11-Pad2): track 4.03 -> 7.15 mm
Changed lines of the file:
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@@
-(kicad_pcb (version 4) (host pcbnew 4.0.6-e0-6349~53~ubuntu16.04.1)
+(kicad_pcb (version 4) (host pcbnew 4.0.4-stable)
   (general
     (links 166)
-    (no_connects 5)
-    (area 56.439999 68.85 172.717143 152.625001)
+    (no_connects 4)
+    (area 56.439999 64.356 172.717143 152.625001)
     (thickness 1.6)
     (drawings 13)
-    (tracks 391)
+    (tracks 393)
     (zones 0)
     (modules 82)
@@
     (0 F.Cu signal)
     (31 B.Cu signal)
-    (32 B.Adhes user)
+    (32 B.Adhes user hide)
     (33 F.Adhes user)
-    (34 B.Paste user)
+    (34 B.Paste user hide)
     (35 F.Paste user)
-    (36 B.SilkS user)
+    (36 B.SilkS user hide)
     (37 F.SilkS user)
-    (38 B.Mask user)
+    (38 B.Mask user hide)
     (39 F.Mask user)
-    (40 Dwgs.User user)
-    (41 Cmts.User user)
-    (42 Eco1.User user)
-    (43 Eco2.User user)
+    (40 Dwgs.User user hide)
+    (41 Cmts.User user hide)
+    (42 Eco1.User user hide)
+    (43 Eco2.User user hide)
     (44 Edge.Cuts user)
     (45 Margin user)
-    (46 B.CrtYd user)
+    (46 B.CrtYd user hide)
     (47 F.CrtYd user)
-    (48 B.Fab user)
+    (48 B.Fab user hide)
     (49 F.Fab user)
   )
@@
     (pad_to_mask_clearance 0.2)
     (aux_axis_origin 0 0)
-    (visible_elements FFFFFF7F)
+    (visible_elements 7FFFFFBF)
     (pcbplotparams
       (layerselection 0x01000_80000001)
@@
       (effects (font (size 1 1) (thickness 0.15)))
     )
-    (fp_text value IR2101 (at 3.81 10.01) (layer F.Fab)
+    (fp_text value IR2101 (at 3.895 6.865) (layer F.Fab)
       (effects (font (size 1 1) (thickness 0.15)))
     )
@@
     (tags "capacitor 1206")
     (attr smd)
-    (fp_text reference C4 (at 5.08 0 90) (layer B.SilkS)
+    (fp_text reference C4 (at -5.325 -0.045 90) (layer B.SilkS)
       (effects (font (size 1 1) (thickness 0.15)) (justify mirror))
     )
-    (fp_text value 10uF (at 0 -2 90) (layer B.Fab)
+    (fp_text value 10uF (at 6.175 -0.145 90) (layer B.Fab)
       (effects (font (size 1 1) (thickness 0.15)) (justify mirror))
     )
@@
     (tags "capacitor 1206")
     (attr smd)
-    (fp_text reference C5 (at 5.08 0 90) (layer B.SilkS)
+    (fp_text reference C5 (at -5.325 0.165 90) (layer B.SilkS)
       (effects (font (size 1 1) (thickness 0.15)) (justify mirror))
     )
-    (fp_text value 0.1uF (at 0 -2 90) (layer B.Fab)
+    (fp_text value 0.1uF (at 6.175 -0.035 90) (layer B.Fab)
       (effects (font (size 1 1) (thickness 0.15)) (justify mirror))
     )
@@
     (tags "capacitor 1206")
     (attr smd)
-    (fp_text reference C6 (at 0 1.75 90) (layer B.SilkS)
+    (fp_text reference C6 (at -4.79 -0.035 90) (layer B.SilkS)
       (effects (font (size 1 1) (thickness 0.15)) (justify mirror))
     )
-    (fp_text value 10uF (at 0 -2 90) (layer B.Fab)
+    (fp_text value 10uF (at 6.21 0.065 90) (layer B.Fab)
       (effects (font (size 1 1) (thickness 0.15)) (justify mirror))
     )
@@
     (tags "capacitor 1206")
     (attr smd)
-    (fp_text reference C7 (at 0 1.75 90) (layer B.SilkS)
+    (fp_text reference C7 (at -5.19 -0.01 90) (layer B.SilkS)
       (effects (font (size 1 1) (thickness 0.15)) (justify mirror))
     )
-    (fp_text value 0.1uF (at 0 -2 90) (layer B.Fab)
+    (fp_text value 0.1uF (at 6.11 -0.01 90) (layer B.Fab)
       (effects (font (size 1 1) (thickness 0.15)) (justify mirror))
     )
@@
     (tags "capacitor 1206")
     (attr smd)
-    (fp_text reference C8 (at 0 1.75 90) (layer B.SilkS)
+    (fp_text reference C8 (at -5.055 -0.11 90) (layer B.SilkS)
       (effects (font (size 1 1) (thickness 0.15)) (justify mirror))
     )
-    (fp_text value 10uF (at 0 -2 90) (layer B.Fab)
+    (fp_text value 10uF (at 6.545 0.09 90) (layer B.Fab)
       (effects (font (size 1 1) (thickness 0.15)) (justify mirror))
     )
@@
     (tags "capacitor 1206")
     (attr smd)
-    (fp_text reference C9 (at 0 1.75 90) (layer B.SilkS)
+    (fp_text reference C9 (at -5.055 -0.135 90) (layer B.SilkS)
       (effects (font (size 1 1) (thickness 0.15)) (justify mirror))
     )
-    (fp_text value 0.1uF (at 0 -2 90) (layer B.Fab)
+    (fp_text value 0.1uF (at 6.645 -0.135 90) (layer B.Fab)
       (effects (font (size 1 1) (thickness 0.15)) (justify mirror))
     )
@@
     (tags "capacitor 1206")
     (attr smd)
-    (fp_text reference C13 (at 0 1.75 180) (layer B.SilkS)
+    (fp_text reference C13 (at -5.225 -0.285 180) (layer B.SilkS)
       (effects (font (size 1 1) (thickness 0.15)) (justify mirror))
     )
-    (fp_text value 100pF (at 0 -2 180) (layer B.Fab)
+    (fp_text value 100pF (at -0.025 3.315 180) (layer B.Fab)
       (effects (font (size 1 1) (thickness 0.15)) (justify mirror))
     )
@@
       (effects (font (size 1 1) (thickness 0.15)) (justify mirror))
     )
-    (fp_text value 100pF (at 0 -2) (layer B.Fab)
+    (fp_text value 100pF (at -6.34 -0.01) (layer B.Fab)
       (effects (font (size 1 1) (thickness 0.15)) (justify mirror))
     )
@@
     (tags "resistor 1206")
     (attr smd)
-    (fp_text reference R7 (at 0 1.85 90) (layer B.SilkS)
+    (fp_text reference R7 (at -4.445 0.005 90) (layer B.SilkS)
       (effects (font (size 1 1) (thickness 0.15)) (justify mirror))
     )
-    (fp_text value 12k (at 0 -1.9 90) (layer B.Fab)
+    (fp_text value 12k (at 5.255 -0.095 90) (layer B.Fab)
       (effects (font (size 1 1) (thickness 0.15)) (justify mirror))
     )
@@
       (effects (font (size 1 1) (thickness 0.15)) (justify mirror))
     )
-    (fp_text value 470k (at 0 -1.9 180) (layer B.Fab)
+    (fp_text value 470k (at -5.225 0.56 180) (layer B.Fab)
       (effects (font (size 1 1) (thickness 0.15)) (justify mirror))
     )
@@
       (effects (font (size 1 1) (thickness 0.15)) (justify mirror))
     )
-    (fp_text value 470k (at 0 -1.9) (layer B.Fab)
+    (fp_text value 470k (at -5.54 0.1) (layer B.Fab)
       (effects (font (size 1 1) (thickness 0.15)) (justify mirror))
     )
@@
     (tags "capacitor 1206")
     (attr smd)
-    (fp_text reference C12 (at 0 1.75) (layer B.SilkS)
+    (fp_text reference C12 (at -5.24 -0.015) (layer B.SilkS)
       (effects (font (size 1 1) (thickness 0.15)) (justify mirror))
     )
-    (fp_text value 100pF (at 0 -2) (layer B.Fab)
+    (fp_text value 100pF (at -0.14 -3.515) (layer B.Fab)
       (effects (font (size 1 1) (thickness 0.15)) (justify mirror))
     )
@@
     (tags "resistor 1206")
     (attr smd)
-    (fp_text reference R27 (at 0 1.85 90) (layer B.SilkS)
+    (fp_text reference R27 (at -4.845 -0.12 90) (layer B.SilkS)
       (effects (font (size 1 1) (thickness 0.15)) (justify mirror))
     )
-    (fp_text value 12k (at 0 -1.9 90) (layer B.Fab)
+    (fp_text value 12k (at 5.155 -0.02 90) (layer B.Fab)
       (effects (font (size 1 1) (thickness 0.15)) (justify mirror))
     )
@@
     (tags "resistor 1206")
     (attr smd)
-    (fp_text reference R29 (at 0 1.85) (layer B.SilkS)
+    (fp_text reference R29 (at -5.14 -0.06) (layer B.SilkS)
       (effects (font (size 1 1) (thickness 0.15)) (justify mirror))
     )
-    (fp_text value 470k (at 0 -1.9) (layer B.Fab)
+    (fp_text value 470k (at 0.06 2.24) (layer B.Fab)
       (effects (font (size 1 1) (thickness 0.15)) (justify mirror))
     )
@@
       (effects (font (size 1 1) (thickness 0.15)))
     )
-    (fp_text value IR2101 (at 3.81 10.01) (layer F.Fab)
+    (fp_text value IR2101 (at 3.895 7.33) (layer F.Fab)
       (effects (font (size 1 1) (thickness 0.15)))
     )
@@
       (effects (font (size 1 1) (thickness 0.15)))
     )
-    (fp_text value IR2101 (at 3.81 10.01) (layer F.Fab)
+    (fp_text value IR2101 (at 3.995 7.495) (layer F.Fab)
       (effects (font (size 1 1) (thickness 0.15)))
     )
@@
   (segment (start 128.905 76.835) (end 128.905 74.335) (width 0.35) (layer F.Cu) (net 1))
   (segment (start 128.905 74.335) (end 130.215 73.025) (width 0.35) (layer F.Cu) (net 1))
-  (segment (start 92.805 73.025) (end 99.06 73.025) (width 0.35) (layer F.Cu) (net 2) (status C00000))
+  (segment (start 92.805 73.025) (end 99.06 73.025) (width 0.35) (layer F.Cu) (net 2))
   (segment (start 64.135 90.17) (end 64.135 87.63) (width 0.35) (layer B.Cu) (net 2))
   (segment (start 64.135 90.17) (end 64.135 92.71) (width 0.35) (layer B.Cu) (net 2))
@@
   (segment (start 116.84 133.985) (end 111.125 128.27) (width 0.35) (layer B.Cu) (net 33))
   (segment (start 128.905 133.985) (end 128.27 133.985) (width 0.6) (layer B.Cu) (net 33))
+  (segment (start 112.395 99.155) (end 115.38 99.155) (width 0.35) (layer B.Cu) (net 34) (status C00000))
+  (segment (start 115.38 99.155) (end 115.475 99.06) (width 0.35) (layer B.Cu) (net 34) (status C00000))
   (segment (start 114.935 102.87) (end 114.935 100.965) (width 0.35) (layer B.Cu) (net 34))
   (segment (start 115.475 100.425) (end 115.475 99.06) (width 0.35) (layer B.Cu) (net 34))
